Commit message: Day 11: Integrated Gazebo Harmonic and spawned VisioBot with physics

File: src/visiobot_core/urdf/visiobot.urdf.xacro (robot description, xacro)
@@ -35,4 +35,10 @@
     </inertial>
   </xacro:macro>
+  <link name="base_footprint"/>
+  <joint name="base_footprint_joint" type="fixed">
+    <parent link="base_footprint"/>
+    <child link="base_link"/>
+    <origin xyz="0 0 0" rpy="0 0 0"/>
+  </joint>
   <link name="base_link">
     <visual>
@@ -138,3 +144,20 @@
     <origin xyz="0.0 0.0 0.075" rpy="0 0 0"/>
   </joint>
+  <gazebo reference="base_link"><material>Gazebo/Blue</material></gazebo>
+  <gazebo reference="right_wheel"><material>Gazebo/Black</material></gazebo>
+  <gazebo reference="left_wheel"><material>Gazebo/Black</material></gazebo>
+  <gazebo reference="camera_link"><material>Gazebo/Red</material></gazebo>
+  <gazebo reference="laser_link"><material>Gazebo/Green</material></gazebo>
+  <gazebo>
+    <plugin filename="gz-sim-diff-drive-system" name="gz::sim::systems::DiffDrive">
+      <left_joint>base_to_left_wheel</left_joint>
+      <right_joint>base_to_right_wheel</right_joint>
+      <wheel_separation>0.35</wheel_separation>
+      <wheel_radius>0.1</wheel_radius>
+      <topic>cmd_vel</topic>
+      <odom_topic>odom</odom_topic>
+      <frame_id>odom</frame_id>
+      <child_frame_id>base_link</child_frame_id>
+    </plugin>
+  </gazebo>
 </robot>

Commit message: Day 12: Added sensor plugins, optical frames, and ros_gz_bridge. LiDAR active.

File: src/visiobot_core/urdf/visiobot.urdf.xacro (robot description, xacro)
@@ -43,15 +43,9 @@
   <link name="base_link">
     <visual>
-      <geometry>
-        <box size="${chassis_length} ${chassis_width} ${chassis_height}"/>
-      </geometry>
-      <material name="blue">
-        <color rgba="0.0 0.2 0.8 1.0"/>
-      </material>
+      <geometry><box size="${chassis_length} ${chassis_width} ${chassis_height}"/></geometry>
+      <material name="blue"><color rgba="0.0 0.2 0.8 1.0"/></material>
     </visual>
     <collision>
-      <geometry>
-        <box size="${chassis_length} ${chassis_width} ${chassis_height}"/>
-      </geometry>
+      <geometry><box size="${chassis_length} ${chassis_width} ${chassis_height}"/></geometry>
     </collision>
     <xacro:box_inertia m="${chassis_mass}" l="${chassis_length}" w="${chassis_width}" h="${chassis_height}"/>
@@ -60,15 +54,9 @@
     <link name="${prefix}_wheel">
       <visual>
-        <geometry>
-          <cylinder radius="${wheel_radius}" length="${wheel_length}"/>
-        </geometry>
-        <material name="black">
-          <color rgba="0.1 0.1 0.1 1.0"/>
-        </material>
+        <geometry><cylinder radius="${wheel_radius}" length="${wheel_length}"/></geometry>
+        <material name="black"><color rgba="0.1 0.1 0.1 1.0"/></material>
       </visual>
       <collision>
-        <geometry>
-          <cylinder radius="${wheel_radius}" length="${wheel_length}"/>
-        </geometry>
+        <geometry><cylinder radius="${wheel_radius}" length="${wheel_length}"/></geometry>
       </collision>
       <xacro:cylinder_inertia m="${wheel_mass}" r="${wheel_radius}" h="${wheel_length}"/>
@@ -84,15 +72,6 @@
   <xacro:wheel prefix="left" y_reflect="1" rpy_val="-1.5708"/>
   <link name="caster_wheel">
-    <visual>
-      <geometry>
-        <sphere radius="0.05"/>
-      </geometry>
-      <material name="black"/>
-    </visual>
-    <collision>
-      <geometry>
-        <sphere radius="0.05"/>
-      </geometry>
-    </collision>
+    <visual><geometry><sphere radius="0.05"/></geometry><material name="black"/></visual>
+    <collision><geometry><sphere radius="0.05"/></geometry></collision>
     <xacro:sphere_inertia m="0.1" r="0.05"/>
   </link>
@@ -104,16 +83,8 @@
   <link name="camera_link">
     <visual>
-      <geometry>
-        <box size="0.05 0.05 0.05"/>
-      </geometry>
-      <material name="red">
-        <color rgba="0.8 0.0 0.0 1.0"/>
-      </material>
+      <geometry><box size="0.05 0.05 0.05"/></geometry>
+      <material name="red"><color rgba="0.8 0.0 0.0 1.0"/></material>
     </visual>
-    <collision>
-      <geometry>
-        <box size="0.05 0.05 0.05"/>
-      </geometry>
-    </collision>
+    <collision><geometry><box size="0.05 0.05 0.05"/></geometry></collision>
     <xacro:box_inertia m="0.1" l="0.05" w="0.05" h="0.05"/>
   </link>
@@ -123,18 +94,16 @@
     <origin xyz="0.18 0.0 0.075" rpy="0 0 0"/>
   </joint>
+  <joint name="camera_optical_joint" type="fixed">
+    <parent link="camera_link"/>
+    <child link="camera_link_optical"/>
+    <origin xyz="0 0 0" rpy="-1.5708 0 -1.5708"/>
+  </joint>
+  <link name="camera_link_optical"></link>
   <link name="laser_link">
     <visual>
-      <geometry>
-        <cylinder radius="0.05" length="0.05"/>
-      </geometry>
-      <material name="green">
-        <color rgba="0.0 0.8 0.0 1.0"/>
-      </material>
+      <geometry><cylinder radius="0.05" length="0.05"/></geometry>
+      <material name="green"><color rgba="0.0 0.8 0.0 1.0"/></material>
     </visual>
-    <collision>
-      <geometry>
-        <cylinder radius="0.05" length="0.05"/>
-      </geometry>
-    </collision>
+    <collision><geometry><cylinder radius="0.05" length="0.05"/></geometry></collision>
     <xacro:cylinder_inertia m="0.2" r="0.05" h="0.05"/>
   </link>
@@ -147,6 +116,53 @@
   <gazebo reference="right_wheel"><material>Gazebo/Black</material></gazebo>
   <gazebo reference="left_wheel"><material>Gazebo/Black</material></gazebo>
-  <gazebo reference="camera_link"><material>Gazebo/Red</material></gazebo>
-  <gazebo reference="laser_link"><material>Gazebo/Green</material></gazebo>
+  <gazebo reference="camera_link">
+    <material>Gazebo/Red</material>
+    <sensor name="camera_sensor" type="camera">
+      <pose>0 0 0 0 0 0</pose>
+      <always_on>true</always_on>
+      <visualize>true</visualize>
+      <update_rate>10.0</update_rate>
+      <camera>
+        <horizontal_fov>1.089</horizontal_fov>
+        <image>
+          <width>640</width>
+          <height>480</height>
+          <format>R8G8B8</format>
+        </image>
+        <clip>
+          <near>0.05</near>
+          <far>8.0</far>
+        </clip>
+      </camera>
+      <topic>/camera/image_raw</topic>
+      <gz_frame_id>camera_link_optical</gz_frame_id>
+    </sensor>
+  </gazebo>
+  <gazebo reference="laser_link">
+    <material>Gazebo/Green</material>
+    <sensor name="laser_sensor" type="gpu_lidar">
+      <pose>0 0 0 0 0 0</pose>
+      <always_on>true</always_on>
+      <visualize>true</visualize>
+      <update_rate>10.0</update_rate>
+      <lidar>
+        <scan>
+          <horizontal>
+            <samples>360</samples>
+            <resolution>1</resolution>
+            <min_angle>-3.14159</min_angle>
+            <max_angle>3.14159</max_angle>
+          </horizontal>
+        </scan>
+        <range>
+          <min>0.12</min>
+          <max>10.0</max>
+          <resolution>0.015</resolution>
+        </range>
+      </lidar>
+      <topic>/scan</topic>
+      <gz_frame_id>laser_link</gz_frame_id>
+    </sensor>
+  </gazebo>
   <gazebo>
     <plugin filename="gz-sim-diff-drive-system" name="gz::sim::systems::DiffDrive">
@@ -158,5 +174,5 @@
       <odom_topic>odom</odom_topic>
       <frame_id>odom</frame_id>
-      <child_frame_id>base_link</child_frame_id>
+      <child_frame_id>base_footprint</child_frame_id>
     </plugin>
   </gazebo>

Commit message: docs: Day13: added bot movements and other wireframes into the virtual world

File: src/visiobot_core/urdf/visiobot.urdf.xacro (robot description, xacro)
@@ -35,9 +35,11 @@
     </inertial>
   </xacro:macro>
+  <!-- base_footprint sits at ground level (z=0). base_link center is raised
+       by wheel_radius so the wheel bottoms touch z=0. -->
   <link name="base_footprint"/>
   <joint name="base_footprint_joint" type="fixed">
     <parent link="base_footprint"/>
     <child link="base_link"/>
-    <origin xyz="0 0 0" rpy="0 0 0"/>
+    <origin xyz="0 0 0.1" rpy="0 0 0"/>
   </joint>
   <link name="base_link">
@@ -51,9 +53,10 @@
     <xacro:box_inertia m="${chassis_mass}" l="${chassis_length}" w="${chassis_width}" h="${chassis_height}"/>
   </link>
+  <!-- Wheel macro: material name includes prefix to avoid duplicate names in Gazebo Harmonic -->
   <xacro:macro name="wheel" params="prefix y_reflect rpy_val">
     <link name="${prefix}_wheel">
       <visual>
         <geometry><cylinder radius="${wheel_radius}" length="${wheel_length}"/></geometry>
-        <material name="black"><color rgba="0.1 0.1 0.1 1.0"/></material>
+        <material name="${prefix}_wheel_black"><color rgba="0.1 0.1 0.1 1.0"/></material>
       </visual>
       <collision>
@@ -71,6 +74,12 @@
   <xacro:wheel prefix="right" y_reflect="-1" rpy_val="1.5708"/>
   <xacro:wheel prefix="left" y_reflect="1" rpy_val="-1.5708"/>
+  <!-- Caster: z offset places its bottom at z=0 relative to base_footprint.
+       base_link center is at z=0.1, so caster center must be at z = -(wheel_radius - caster_radius)
+       = -(0.1 - 0.05) = -0.05 from base_link. -->
   <link name="caster_wheel">
-    <visual><geometry><sphere radius="0.05"/></geometry><material name="black"/></visual>
+    <visual>
+      <geometry><sphere radius="0.05"/></geometry>
+      <material name="caster_black"><color rgba="0.1 0.1 0.1 1.0"/></material>
+    </visual>
     <collision><geometry><sphere radius="0.05"/></geometry></collision>
     <xacro:sphere_inertia m="0.1" r="0.05"/>
@@ -171,9 +180,15 @@
       <wheel_separation>0.35</wheel_separation>
       <wheel_radius>0.1</wheel_radius>
-      <topic>cmd_vel</topic>
-      <odom_topic>odom</odom_topic>
+      <topic>/cmd_vel</topic>
+      <odom_topic>/odom</odom_topic>
+      <tf_topic>/tf</tf_topic>
       <frame_id>odom</frame_id>
       <child_frame_id>base_footprint</child_frame_id>
     </plugin>
+    <plugin filename="gz-sim-joint-state-publisher-system" name="gz::sim::systems::JointStatePublisher">
+      <topic>/joint_states</topic>
+      <joint_name>base_to_left_wheel</joint_name>
+      <joint_name>base_to_right_wheel</joint_name>
+    </plugin>
   </gazebo>
 </robot>

Commit message: fix: NAV2 initial

File: src/visiobot_core/urdf/visiobot.urdf.xacro (robot description, xacro)
@@ -45,6 +45,31 @@
   <link name="base_link">
     <visual>
-      <geometry><box size="${chassis_length} ${chassis_width} ${chassis_height}"/></geometry>
-      <material name="blue"><color rgba="0.0 0.2 0.8 1.0"/></material>
+      <geometry><box size="0.38 0.28 0.06"/></geometry>
+      <material name="car_body"><color rgba="0.15 0.15 0.18 1.0"/></material>
+    </visual>
+    <visual>
+      <origin xyz="0.14 0 -0.01" rpy="0 0 0"/>
+      <geometry><box size="0.12 0.26 0.04"/></geometry>
+      <material name="car_hood"><color rgba="0.85 0.1 0.1 1.0"/></material>
+    </visual>
+    <visual>
+      <origin xyz="-0.02 0 0.065" rpy="0 0 0"/>
+      <geometry><box size="0.14 0.24 0.07"/></geometry>
+      <material name="car_cabin"><color rgba="0.1 0.15 0.3 1.0"/></material>
+    </visual>
+    <visual>
+      <origin xyz="-0.18 0 0.06" rpy="0 0 0"/>
+      <geometry><box size="0.02 0.26 0.03"/></geometry>
+      <material name="car_spoiler"><color rgba="0.95 0.85 0.1 1.0"/></material>
+    </visual>
+    <visual>
+      <origin xyz="0.2 0 -0.02" rpy="0 0 0"/>
+      <geometry><box size="0.04 0.28 0.03"/></geometry>
+      <material name="car_bumper_front"><color rgba="0.7 0.7 0.75 1.0"/></material>
+    </visual>
+    <visual>
+      <origin xyz="-0.2 0 -0.02" rpy="0 0 0"/>
+      <geometry><box size="0.04 0.28 0.03"/></geometry>
+      <material name="car_bumper_rear"><color rgba="0.7 0.7 0.75 1.0"/></material>
     </visual>
     <collision>
